File: PIC24 USB/_autosave-PIC24_USB_IR_Transmitter.kicad_pcb (KiCad board)
At the start: 2 copper layers, 53 parts, among them CON1 USB-MINI-B, P1 CONN_6, P2 CONN_4, P3 CONN_4, P4 CONN_8, P5 CONN_4, P6 CONN_1, P7 CONN_8, P8 CONN_8X2, Q1 2N7002, Q2 MOSFET_N, Q3 MOSFET_N, Q4 MOSFET_N, Q5 MOSFET_N, Q6 MOSFET_N, Q7 MOSFET_N, Q8 MOSFET_N, U1 PIC24FJXXXGB106, U2 LM1117_SOT223_3V3, U3 50mm_5x7_Dot_Matrix_Led_Displ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, U4 MCP48X2, X1 CRYSTAL_12MHZ

Commit message: fixed some oopsies
Parts:
- removed 10u1, 10u2: C, SM1206
- added R14: 0R, SMD_Packages:SMD-1206, F.Cu at (28.5, 35.0)
- added R15: 100K, SMD_Packages:SMD-0603_r, F.Cu at (48.5, 42.2)
- added X2: 32khz, Crystals:Crystal_Round_Horizontal_3mm_BigPad, F.Cu at (64.7, 45.9)
- C5, C6: value 100n -> ?
- D1: value POWER_LED -> LED_POWER
- P6: footprint Pin_Headers:Pin_Header_Straight_1x01 -> Symbols:Symbol_OSHW-Logo_CopperTop
- moved P6 58.1 mm to (86.7, 17.8)
- moved P3 57.8 mm to (40.8, 55.2)
- moved R13 52.6 mm to (38.5, 48.0)
- moved P2 49.3 mm to (42.5, 16.5)
- moved P7 49.0 mm to (87.7, 38.0), turned to 270 degrees
- moved U4 48.2 mm to (42.1, 44.5), turned to 180 degrees
- moved D1 44.1 mm to (26.2, 58.8)
- moved R1 44.1 mm to (30.1, 59.2)
- moved U2 41.1 mm to (28.8, 49.8)
- moved C13 41.1 mm to (28.1, 55.8)
- moved P5 40.8 mm to (15.5, 23.2), turned to 270 degrees
- moved C1 37.3 mm to (20.6, 53.9)
- moved D3 35.9 mm to (72.8, 57.0), turned to 0 degrees
- moved C2 35.8 mm to (44.8, 44.2), turned to 270 degrees
- moved R4 34.3 mm to (67.3, 57.0)
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Connections:
- net /MCUSection/RP14 renamed /MCUSection/AN14/RP14/RB14
- net /MCUSection/RP29 renamed /MCUSection/AN15/RP29/RB15
- net Net-(U1-Pad24) renamed /MCUSection/AN11/RB11
- net Net-(U1-Pad27) renamed /MCUSection/AN12/RB12
- C5 pad 1: /VUSB -> /MCUSection/SOSCI
- C6 pad 1: GND -> /MCUSection/SOSCO
- C6 pad 2: +5V -> GND
- CON1 pad 1: +5V -> /VIN
- CON1 pad 2: D- -> /MCUSection/D-
- CON1 pad 3: D+ -> /MCUSection/D+
- D2 pad 2: Net-(D2-Pad2) -> GND
- P1 pad 1: ~MCLR~ -> Net-(P1-Pad1)
- P1 pad 2: +3.3V -> PGC
- P1 pad 3: GND -> PGD
- P1 pad 4: PGD -> GND
- P1 pad 5: PGC -> +3.3V
- P1 pad 6: Net-(P1-Pad6) -> ~MCLR~
- Q1 pad G: IR_LED -> /MCUSection/AN13/RB1
- R13 pad 1: /~LDAC~ -> /MCUSection/AN10/RB10
- R3 pad 1: /USER_LED -> /MCUSection/RF1
- U1 pad 21: Net-(U1-Pad21) -> /MCUSection/AN8/RP8/RB8
- U1 pad 22: Net-(U1-Pad22) -> /MCUSection/AN9/RP9/RB9
- U1 pad 23: Net-(U1-Pad23) -> /MCUSection/AN10/RB10
- U1 pad 28: Net-(U1-Pad28) -> /MCUSection/AN13/RB1
- U1 pad 33: Net-(U1-Pad33) -> /MCUSection/RP16/RF3
- U1 pad 34: Net-(U1-Pad34) -> /MCUSection/VBUS_SENSE
- U1 pad 35: Net-(U1-Pad35) -> +3.3V
- U1 pad 36: Net-(U1-Pad36) -> /MCUSection/D-
- U1 pad 37: Net-(U1-Pad37) -> /MCUSection/D+
- U1 pad 47: Net-(U1-Pad47) -> /MCUSection/SOSCI
- U1 pad 48: Net-(U1-Pad48) -> /MCUSection/SOSCO
- U1 pad 58: Net-(U1-Pad58) -> ~LCD_RESET~
- U1 pad 59: Net-(U1-Pad59) -> /MCUSection/RF1
- U4 pad 2: /~CS~DAC -> /MCUSection/RP16/RF3
- U4 pad 3: /SCKDAC -> /MCUSection/AN9/RP9/RB9
- U4 pad 4: /SDIDAC -> /MCUSection/AN8/RP8/RB8
- U4 pad 5: /~LDAC~ -> /MCUSection/AN10/RB10
Routing:
- net +5V: track 57.4 -> 257.3 mm, vias 0 -> 1
- net +3.3V: track 125.2 -> 223.9 mm, vias 0 -> 2
- net GND: track 73.2 -> 153.8 mm, vias 3 -> 9
- net SCL: track 38.5 -> 97.6 mm, vias 0 -> 2
- net SDA: track 45.1 -> 93.2 mm, vias 0 -> 4
- net Net-(R10-Pad2): track 2.76 -> 48.2 mm
- net /MCUSection/AN10/RB10: track 0.00 -> 42.2 mm, vias 0 -> 2
- net /MCUSection/D+: track 0.00 -> 36.1 mm
- net /MCUSection/D-: track 0.00 -> 35.7 mm
- net /MCUSection/PORTD6: track 66.7 -> 39.4 mm
- net /Dot Matrix Sheet/C2: track 74.6 -> 47.3 mm
- net /MCUSection/PORTD4: track 97.3 -> 70.9 mm
- net ~LCD_RESET~: track 0.00 -> 26.4 mm
- net /MCUSection/PORTD2: track 97.1 -> 71.4 mm
- net /MCUSection/PORTD5: track 89.9 -> 64.3 mm
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Other:
- board outline added: 101 x 47.6 mm
- net class POWER added: clearance 0.15, trace_width 0.254, via_dia 0.889, via_drill 0.635
