File: PIC24 USB/MCU.sch (KiCad schematic (older format))
At the start: 16 parts, among them U1 PIC24FJXXXGB106, X1 CRYSTAL_12MHZ, X2 32khz

Commit message: Updated
Parts:
- C10, C11, C12, C3, C4, C5, C6, C7, C8, C9: symbol C -> C-RESCUE-PIC24_USB_IR_Transmitter
- R15, R2, R7: symbol R -> R-RESCUE-PIC24_USB_IR_Transmitter
Changed lines of the file:
@@
 EESchema Schematic File Version 2
+LIBS:PIC24_USB_IR_Transmitter-rescue
 LIBS:power
 LIBS:device
@@
 LIBS:led_hele
 LIBS:PIC24_USB_IR_Transmitter-cache
-EELAYER 24 0
+EELAYER 25 0
 EELAYER END
 $Descr A4 11693 8268
@@
 ~MCLR
 $Comp
-L GND #PWR048
+L GND-RESCUE-PIC24_USB_IR_Transmitter #PWR048
 U 1 1 53DA26E1
 P 1750 3500
@@
 $EndComp
 $Comp
-L GND #PWR049
+L GND-RESCUE-PIC24_USB_IR_Transmitter #PWR049
 U 1 1 53DA26EE
 P 2200 5150
@@
 $EndComp
 $Comp
-L GND #PWR050
+L GND-RESCUE-PIC24_USB_IR_Transmitter #PWR050
 U 1 1 53DA26F4
 P 8050 3300
@@
 $EndComp
 $Comp
-L C C9
+L C-RESCUE-PIC24_USB_IR_Transmitter C9
 U 1 1 53DA330C
 P 9050 2650
+AR Path="/53DA330C" Ref="C9"  Part="1"
+AR Path="/53DA26B9/53DA330C" Ref="C9"  Part="1"
 F 0 "C9" H 9050 2750 40  0000 L CNN
 F 1 "22p" H 9056 2565 40  0000 L CNN
@@
 $EndComp
 $Comp
-L C C10
+L C-RESCUE-PIC24_USB_IR_Transmitter C10
 U 1 1 53DA3319
 P 9050 3250
+AR Path="/53DA3319" Ref="C10"  Part="1"
+AR Path="/53DA26B9/53DA3319" Ref="C10"  Part="1"
 F 0 "C10" H 9050 3350 40  0000 L CNN
 F 1 "22p" H 9056 3165 40  0000 L CNN
@@
 $EndComp
 $Comp
-L GND #PWR055
+L GND-RESCUE-PIC24_USB_IR_Transmitter #PWR055
 U 1 1 53DA331F
 P 9550 3050
@@
 $EndComp
 $Comp
-L C C3
+L C-RESCUE-PIC24_USB_IR_Transmitter C3
 U 1 1 53DA3435
 P 1450 4150
+AR Path="/53DA3435" Ref="C3"  Part="1"
+AR Path="/53DA26B9/53DA3435" Ref="C3"  Part="1"
 F 0 "C3" H 1450 4250 40  0000 L CNN
 F 1 "100n" H 1456 4065 40  0000 L CNN
@@
 $EndComp
 $Comp
-L GND #PWR056
+L GND-RESCUE-PIC24_USB_IR_Transmitter #PWR056
 U 1 1 53DA3460
 P 1450 4450
@@
 $EndComp
 $Comp
-L C C4
+L C-RESCUE-PIC24_USB_IR_Transmitter C4
 U 1 1 53DA3506
 P 2200 4850
+AR Path="/53DA3506" Ref="C4"  Part="1"
+AR Path="/53DA26B9/53DA3506" Ref="C4"  Part="1"
 F 0 "C4" H 2200 4950 40  0000 L CNN
 F 1 "100n" H 2206 4765 40  0000 L CNN
@@
 $EndComp
 $Comp
-L C C7
+L C-RESCUE-PIC24_USB_IR_Transmitter C7
 U 1 1 53DA35D7
 P 1750 3200
+AR Path="/53DA35D7" Ref="C7"  Part="1"
+AR Path="/53DA26B9/53DA35D7" Ref="C7"  Part="1"
 F 0 "C7" H 1750 3300 40  0000 L CNN
 F 1 "100n" H 1756 3115 40  0000 L CNN
@@
 $EndComp
 $Comp
-L C C8
+L C-RESCUE-PIC24_USB_IR_Transmitter C8
 U 1 1 53DA3748
 P 8050 2950
+AR Path="/53DA3748" Ref="C8"  Part="1"
+AR Path="/53DA26B9/53DA3748" Ref="C8"  Part="1"
 F 0 "C8" H 8050 3050 40  0000 L CNN
 F 1 "100n" H 8056 2865 40  0000 L CNN
@@
 $EndComp
 $Comp
-L C C12
+L C-RESCUE-PIC24_USB_IR_Transmitter C12
 U 1 1 53DC00CE
 P 8350 4700
+AR Path="/53DC00CE" Ref="C12"  Part="1"
+AR Path="/53DA26B9/53DC00CE" Ref="C12"  Part="1"
 F 0 "C12" H 8350 4800 40  0000 L CNN
 F 1 "10u" H 8356 4615 40  0000 L CNN
@@
 $EndComp
 $Comp
-L GND #PWR058
+L GND-RESCUE-PIC24_USB_IR_Transmitter #PWR058
 U 1 1 53DC0153
 P 8350 4950
@@
 PGED
 $Comp
-L R R7
+L R-RESCUE-PIC24_USB_IR_Transmitter R7
 U 1 1 53DEB244
 P 1350 2900
@@
 $EndComp
 $Comp
-L R R2
+L R-RESCUE-PIC24_USB_IR_Transmitter R2
 U 1 1 53DEB251
 P 1000 2550
@@
 $EndComp
 $Comp
-L C C11
+L C-RESCUE-PIC24_USB_IR_Transmitter C11
 U 1 1 53DEB257
 P 1000 3200
+AR Path="/53DEB257" Ref="C11"  Part="1"
+AR Path="/53DA26B9/53DEB257" Ref="C11"  Part="1"
 F 0 "C11" H 1000 3300 40  0000 L CNN
 F 1 "100n" H 1006 3115 40  0000 L CNN
@@
 $EndComp
 $Comp
-L GND #PWR059
+L GND-RESCUE-PIC24_USB_IR_Transmitter #PWR059
 U 1 1 53DEB25D
 P 1000 3500
@@
 $EndComp
 $Comp
-L R R15
+L R-RESCUE-PIC24_USB_IR_Transmitter R15
 U 1 1 53EB0F03
 P 8450 2100
@@
 $EndComp
 $Comp
-L C C5
+L C-RESCUE-PIC24_USB_IR_Transmitter C5
 U 1 1 53F4D6C5
 P 9400 3600
+AR Path="/53F4D6C5" Ref="C5"  Part="1"
+AR Path="/53DA26B9/53F4D6C5" Ref="C5"  Part="1"
 F 0 "C5" H 9400 3700 40  0000 L CNN
 F 1 "?" H 9406 3515 40  0000 L CNN
@@
 $EndComp
 $Comp
-L C C6
+L C-RESCUE-PIC24_USB_IR_Transmitter C6
 U 1 1 53F4D77C
 P 9400 4300
+AR Path="/53F4D77C" Ref="C6"  Part="1"
+AR Path="/53DA26B9/53F4D77C" Ref="C6"  Part="1"
 F 0 "C6" H 9400 4400 40  0000 L CNN
 F 1 "?" H 9406 4215 40  0000 L CNN
@@
 $EndComp
 $Comp
-L GND #PWR063
+L GND-RESCUE-PIC24_USB_IR_Transmitter #PWR063
 U 1 1 53F4D7BA
 P 9800 4000
