File: PIC24 USB/PIC24_USB_IR_Transmitter.sch (KiCad schematic (older format))
At the start: 35 parts, among them CON1 USB-MINI-B, P1 CONN_6, P2 CONN_4, P3 CONN_4, P4 CONN_8, P5 CONN_4, P6 CONN_1, P7 CONN_8, P8 CONN_8X2, Q1 2N7002, U2 LM1117_SOT223_3V3, U4 MCP48X2, U5 MCP9700, U6 24C16, U7 TCN75

Commit message: Updated
Parts:
- C1: symbol CP -> CP-RESCUE-PIC24_USB_IR_Transmitter
- C13, C14, C15, C16, C2: symbol C -> C-RESCUE-PIC24_USB_IR_Transmitter
- D1, D2, D3: symbol LED -> LED-RESCUE-PIC24_USB_IR_Transmitter
- R1, R13, R14, R18, R19, R20, R21, R3, R4, R5, R6: symbol R -> R-RESCUE-PIC24_USB_IR_Transmitter
Changed lines of the file:
@@
 EESchema Schematic File Version 2
+LIBS:PIC24_USB_IR_Transmitter-rescue
 LIBS:power
 LIBS:device
@@
 LIBS:led_hele
 LIBS:PIC24_USB_IR_Transmitter-cache
-EELAYER 24 0
+EELAYER 25 0
 EELAYER END
 $Descr A4 11693 8268
@@
 Connection ~ 950  3150
 $Comp
-L GND #PWR01
+L GND-RESCUE-PIC24_USB_IR_Transmitter #PWR01
 U 1 1 52D43B6B
 P 2200 3350
@@
 $EndComp
 $Comp
-L CP C1
+L CP-RESCUE-PIC24_USB_IR_Transmitter C1
 U 1 1 52D43BC9
 P 1200 1350
@@
 $EndComp
 $Comp
-L GND #PWR04
+L GND-RESCUE-PIC24_USB_IR_Transmitter #PWR04
 U 1 1 52D43BDC
 P 1200 1650
@@
 D-
 $Comp
-L C C2
+L C-RESCUE-PIC24_USB_IR_Transmitter C2
 U 1 1 52D44076
 P 8850 3950
@@
 	1750 6050 1750 6300
 $Comp
-L GND #PWR05
+L GND-RESCUE-PIC24_USB_IR_Transmitter #PWR05
 U 1 1 52D450A4
 P 1750 6300
@@
 ~MCLR~
 $Comp
-L GND #PWR06
+L GND-RESCUE-PIC24_USB_IR_Transmitter #PWR06
 U 1 1 52D45877
 P 10800 4000
@@
 	10800 3900 10800 4000
 $Comp
-L R R4
+L R-RESCUE-PIC24_USB_IR_Transmitter R4
 U 1 1 52D4596A
 P 10800 2750
@@
 $EndComp
 $Comp
-L LED D3
+L LED-RESCUE-PIC24_USB_IR_Transmitter D3
 U 1 1 52D45985
 P 10800 3250
@@
 	5250 1750 5550 1750
 $Comp
-L R R3
+L R-RESCUE-PIC24_USB_IR_Transmitter R3
 U 1 1 52D45E25
 P 4450 5450
@@
 $EndComp
 $Comp
-L LED D2
+L LED-RESCUE-PIC24_USB_IR_Transmitter D2
 U 1 1 52D45E2B
 P 4450 5950
@@
 	4450 4200 4450 5200
 $Comp
-L R R1
+L R-RESCUE-PIC24_USB_IR_Transmitter R1
 U 1 1 52D45EB1
 P 1650 1200
@@
 $EndComp
 $Comp
-L LED D1
+L LED-RESCUE-PIC24_USB_IR_Transmitter D1
 U 1 1 52D45EB7
 P 1650 1700
@@
 	1650 850  1650 950
 $Comp
-L GND #PWR08
+L GND-RESCUE-PIC24_USB_IR_Transmitter #PWR08
 U 1 1 52D45EC1
 P 1650 1950
@@
 $EndComp
 $Comp
-L GND #PWR010
+L GND-RESCUE-PIC24_USB_IR_Transmitter #PWR010
 U 1 1 52D4649C
 P 8350 3450
@@
 $EndComp
 $Comp
-L GND #PWR011
+L GND-RESCUE-PIC24_USB_IR_Transmitter #PWR011
 U 1 1 52D464B4
 P 3700 5050
@@
 $EndComp
 $Comp
-L R R5
+L R-RESCUE-PIC24_USB_IR_Transmitter R5
 U 1 1 52D469B5
 P 3800 4500
@@
 Connection ~ 3800 4900
 $Comp
-L R R6
+L R-RESCUE-PIC24_USB_IR_Transmitter R6
 U 1 1 52D46B46
 P 3950 4500
@@
 $EndComp
 $Comp
-L GND #PWR015
+L GND-RESCUE-PIC24_USB_IR_Transmitter #PWR015
 U 1 1 52D8FECF
 P 1300 7650
@@
 $EndComp
 $Comp
-L GND #PWR019
+L GND-RESCUE-PIC24_USB_IR_Transmitter #PWR019
 U 1 1 53DC0948
 P 5450 7300
@@
 	5450 7200 5450 7300
 $Comp
-L GND #PWR020
+L GND-RESCUE-PIC24_USB_IR_Transmitter #PWR020
 U 1 1 53DC0A13
 P 6000 7300
@@
 $EndComp
 $Comp
-L C C13
+L C-RESCUE-PIC24_USB_IR_Transmitter C13
 U 1 1 53DC0A22
 P 6000 6950
@@
 $EndComp
 $Comp
-L GND #PWR024
+L GND-RESCUE-PIC24_USB_IR_Transmitter #PWR024
 U 1 1 53EA6786
 P 4400 4000
@@
 	3100 850  3100 1700
 $Comp
-L GND #PWR025
+L GND-RESCUE-PIC24_USB_IR_Transmitter #PWR025
 U 1 1 53EA8972
 P 3450 2000
@@
 	9550 3950 9550 4750
 $Comp
-L GND #PWR028
+L GND-RESCUE-PIC24_USB_IR_Transmitter #PWR028
 U 1 1 53EB3792
 P 9550 4750
@@
 Connection ~ 8100 3950
 $Comp
-L GND #PWR029
+L GND-RESCUE-PIC24_USB_IR_Transmitter #PWR029
 U 1 1 53EB8094
 P 9800 4600
@@
 VOUTB
 $Comp
-L GND #PWR030
+L GND-RESCUE-PIC24_USB_IR_Transmitter #PWR030
 U 1 1 53EB8CF7
 P 9350 5300
@@
 $EndComp
 $Comp
-L R R13
+L R-RESCUE-PIC24_USB_IR_Transmitter R13
 U 1 1 53EB8D1B
 P 9350 4950
@@
 IR_LED
 $Comp
-L R R14
+L R-RESCUE-PIC24_USB_IR_Transmitter R14
 U 1 1 53EF297E
 P 2250 2250
@@
 replace with polyfuse\nor ferrite if needed
 $Comp
-L GND #PWR033
+L GND-RESCUE-PIC24_USB_IR_Transmitter #PWR033
 U 1 1 53EFE3A1
 P 4450 6200
@@
 VOUTA
 $Comp
-L GND #PWR034
+L GND-RESCUE-PIC24_USB_IR_Transmitter #PWR034
 U 1 1 52D43B2E
 P 950 3350
@@
 VOUT_TEMP_SEMS
 $Comp
-L GND #PWR035
+L GND-RESCUE-PIC24_USB_IR_Transmitter #PWR035
 U 1 1 53ECDE47
 P 6700 6150
@@
 $EndComp
 $Comp
-L C C14
+L C-RESCUE-PIC24_USB_IR_Transmitter C14
 U 1 1 53ECF8B3
 P 6700 5850
@@
 $EndComp
 $Comp
-L GND #PWR037
+L GND-RESCUE-PIC24_USB_IR_Transmitter #PWR037
 U 1 1 54641AA4
 P 2500 4700
@@
 	3200 4300 3250 4300
 $Comp
-L GND #PWR039
+L GND-RESCUE-PIC24_USB_IR_Transmitter #PWR039
 U 1 1 54642FFC
 P 3250 4050
@@
 	3250 4000 3250 4050
 $Comp
-L GND #PWR040
+L GND-RESCUE-PIC24_USB_IR_Transmitter #PWR040
 U 1 1 54643197
 P 1750 4200
@@
 Connection ~ 1750 4100
 $Comp
-L R R18
+L R-RESCUE-PIC24_USB_IR_Transmitter R18
 U 1 1 546436E1
 P 1300 3900
@@
 $EndComp
 $Comp
-L R R19
+L R-RESCUE-PIC24_USB_IR_Transmitter R19
 U 1 1 5464377C
 P 1300 4500
@@
 $EndComp
 $Comp
-L GND #PWR041
+L GND-RESCUE-PIC24_USB_IR_Transmitter #PWR041
 U 1 1 54643B72
 P 1300 4800
@@
 	1300 3650 1300 3600
 $Comp
-L C C15
+L C-RESCUE-PIC24_USB_IR_Transmitter C15
 U 1 1 5464427C
 P 1650 3900
@@
 	3600 6150 3700 6150
 $Comp
-L GND #PWR043
+L GND-RESCUE-PIC24_USB_IR_Transmitter #PWR043
 U 1 1 5464ADEE
 P 3700 6700
@@
 $EndComp
 $Comp
-L GND #PWR044
+L GND-RESCUE-PIC24_USB_IR_Transmitter #PWR044
 U 1 1 5464AED8
 P 2550 6450
@@
 Connection ~ 3700 6550
 $Comp
-L R R20
+L R-RESCUE-PIC24_USB_IR_Transmitter R20
 U 1 1 54651E19
 P 2100 6150
@@
 $EndComp
 $Comp
-L R R21
+L R-RESCUE-PIC24_USB_IR_Transmitter R21
 U 1 1 54651E1F
 P 2100 6750
@@
 $EndComp
 $Comp
-L GND #PWR046
+L GND-RESCUE-PIC24_USB_IR_Transmitter #PWR046
 U 1 1 54651E25
 P 2100 7050
@@
 	2100 5900 2100 5850
 $Comp
-L C C16
+L C-RESCUE-PIC24_USB_IR_Transmitter C16
 U 1 1 54651E39
 P 2450 6150
