File: USB IR Transmitter/pic18_USB_IR_Transmitter.sch (KiCad schematic (older format))
At the start: 26 parts, among them CON1 USB-MINI-B, P1 CONN_6, P2 CONN_4, P3 CONN_6, P4 CONN_6, P5 CONN_4, P6 CONN_1, P7 CONN_8, Q1 2N7002, U1 1586-PIC18F4550-I/PT, X1 12Mhz

Commit message: fixed footprint name error in PIC18f board, rerouted board layout
Parts:
- C1: footprint (none) -> Capacitors_Tantalum_SMD:TantalC_SizeC_EIA-6032_Reflow
- C2, C3, C4, C5, C6: footprint (none) -> Capacitors_SMD:C_0603
- CON1: footprint (none) -> Connect:USB_Mini-B
- D1, D2: footprint (none) -> LEDs:LED-0603
- D3: footprint (none) -> LEDs:LED-3MM
- P1: footprint (none) -> Pin_Headers:Pin_Header_Angled_1x06
- P2, P5: footprint (none) -> Pin_Headers:Pin_Header_Straight_1x04
- P3, P4: footprint (none) -> Pin_Headers:Pin_Header_Straight_1x06
- P6: footprint (none) -> Pin_Headers:Pin_Header_Straight_1x01
- P7: footprint (none) -> midas_lcd:midas_i2c_lcd
- Q1: footprint (none) -> SMD_Packages:SOT-23-GDS
- R1, R2, R3, R5, R6: footprint (none) -> Resistors_SMD:R_0603
- R4: footprint (none) -> Resistors_SMD:R_1206
- U1: footprint bittenbybytes/axylf -> QFP:LQFP-44_10x10mm_Pitch0.8mm
- X1: footprint (none) -> Crystals_Oscillators_SMD:Q_49U3HMS
